Commit message: Reflect cameras on the real robot

File: rae_description/urdf/rae.urdf.xacro (robot description, xacro)
@@ -5,4 +5,5 @@
   <xacro:arg name="namespace" default="" />
   <xacro:include filename="inertial_moment_calc.xacro"/>
+  <xacro:include filename="camera.urdf.xacro"/>
   <xacro:include filename="rae_ros2_control.urdf.xacro"/>
   <xacro:property name="deg_to_rad" value="0.01745329251994329577" />
@@ -301,98 +302,8 @@
   <xacro:rae_ros2_control sim_mode="$(arg sim_mode)" namespace="$(arg namespace)" />
   <xacro:if value="$(arg sim_mode)">
-    <link name="rae_rgb_camera_sim_frame">
-      <xacro:body mass="0.00001" d="0.0000010" h="0.000003" w="0.00003">
-        <origin xyz="0.0 0.0 0.0" rpy="0.0 0.0 0.0"/>
-      </xacro:body>
-    </link>
-    <joint name="rae_rgb_camera_sim_frame_joint" type="fixed">
-      <origin xyz="0.0 0 0" rpy="${pi/2} ${-pi/2} 0.0"/>
-      <parent link="rae_rgb_camera_optical_frame"/>
-      <child link="rae_rgb_camera_sim_frame"/>
-    </joint>
-    <gazebo reference="rae_rgb_camera_sim_frame">
-      <sensor type="camera" name="rae_rgb_camera">
-        <always_on>true</always_on>
-        <update_rate>30.0</update_rate>
-        <topic>/rae/right/image_raw</topic>
-        <ignition_frame_id>rae_rgb_camera_optical_frame</ignition_frame_id>
-        <camera>
-          <horizontal_fov>${105.0/180.0*pi}</horizontal_fov>
-          <image>
-            <width>320</width>
-            <height>240</height>
-          </image>
-          <clip>
-            <near>0.1</near>
-            <far>100</far>
-          </clip>
-          <noise>
-            <type>gaussian</type>
-            <mean>0.0</mean>
-            <stddev>0.007</stddev>
-          </noise>
-        </camera>
-      </sensor>
-      <plugin filename="ignition-gazebo-sensors-system" name="ignition::gazebo::systems::Sensors">
-        <engine>ogre2</engine>
-      </plugin>
-    </gazebo>
-    <link name="rae_stereo_front_frame">
-      <xacro:body mass="0.00001" d="0.00001" h="0.000003" w="0.00001">
-        <origin xyz="0.0 0.0 0.0" rpy="0.0 0.0 0.0"/>
-      </xacro:body>
-    </link>
-    <joint name="rae_stereo_front_frame_joint" type="fixed">
-      <origin xyz="${0.0208282} 0.0 0.0100195" rpy="0.0 ${-30.0/180*pi} 0.0"/>
-      <parent link="base_link"/>
-      <child link="rae_stereo_front_frame"/>
-    </joint>
-    <gazebo reference="rae_stereo_front_frame">
-      <sensor name="front_depth_camera" type="depth_camera">
-        <update_rate>15.0</update_rate>
-        <topic>/rae/stereo_front/image_raw</topic>
-        <ignition_frame_id>rae_stereo_front_frame</ignition_frame_id>
-        <camera>
-          <horizontal_fov>${60.0/180.0*pi}</horizontal_fov>
-          <image>
-            <width>320</width>
-            <height>240</height>
-          </image>
-          <clip>
-            <near>0.2</near>
-            <far>6.0</far>
-          </clip>
-        </camera>
-      </sensor>
-    </gazebo>
-    <link name="rae_stereo_rear_frame">
-      <xacro:body mass="0.00001" d="0.00001" h="0.00001" w="0.00001">
-        <origin xyz="0.0 0.0 0.0" rpy="0.0 0.0 0.0"/>
-      </xacro:body>
-    </link>
-    <joint name="rae_stereo_rear_frame_joint" type="fixed">
-      <origin xyz="${-0.0822282} 0.0 0.0100195" rpy="0.0 ${-30.0/180*pi} ${pi}"/>
-      <parent link="base_link"/>
-      <child link="rae_stereo_rear_frame"/>
-    </joint>
-    <gazebo reference="rae_stereo_rear_frame">
-      <sensor name="rear_depth_camera" type="depth_camera">
-        <update_rate>15.0</update_rate>
-        <topic>/rae/stereo_back/image_raw</topic>
-        <vizualize>true</vizualize>
-        <ignition_frame_id>rae_stereo_rear_frame</ignition_frame_id>
-        <camera>
-          <horizontal_fov>${60.0/180.0*pi}</horizontal_fov>
-          <image>
-            <width>320</width>
-            <height>240</height>
-          </image>
-          <clip>
-            <near>0.2</near>
-            <far>6.0</far>
-          </clip>
-        </camera>
-      </sensor>
-    </gazebo>
+    <xacro:rae_mono_camera camera_name="right" ns="$(arg namespace)" enable_depth="true" />
+    <xacro:rae_mono_camera camera_name="left_back" ns="$(arg namespace)" enable_depth="true" />
+    <!-- Uncomment when RGB camera is available on real robot -->
+    <!-- <xacro:rae_rgb_camera camera_name="rgb" ns="$(arg namespace)" /> -->
   </xacro:if>
 </robot>
